File: ai03 pcb guide.sch (KiCad schematic (older format))
At the start: 24 parts, among them SW1 SW_Push, U1 ATmega32U4-AU, Y1 16MHz

Commit message: routed
Parts:
- renumbered D3 to D2, D2 to D3, MX3 to MX2, MX2 to MX3
Connections:
- net COL0: now also U1.29 (PB5)
- net COL1: now also U1.28 (PB4)
- net ROW0: now also U1.27 (PD7)
- net ROW1: now also U1.30 (PB6)
Changed lines of the file:
@@
 	6950 3250 7050 3250
 $Comp
-L MX_Alps_Hybrid:MX-NoLED MX3
+L MX_Alps_Hybrid:MX-NoLED MX2
 U 1 1 612BFDD5
 P 7700 3100
-F 0 "MX3" H 7733 3323 60  0000 C CNN
+F 0 "MX2" H 7733 3323 60  0000 C CNN
 F 1 "MX-NoLED" H 7733 3249 20  0000 C CNN
 F 2 "MX_Alps_Hybrid:MX-1U" H 7075 3075 60  0001 C CNN
@@
 $EndComp
 $Comp
-L Device:D_Small D3
+L Device:D_Small D2
 U 1 1 612C056B
 P 7550 3350
-F 0 "D3" V 7596 3280 50  0000 R CNN
+F 0 "D2" V 7596 3280 50  0000 R CNN
 F 1 "SOD-123" V 7505 3280 50  0000 R CNN
 F 2 "Diode_SMD:D_SOD-123" V 7550 3350 50  0001 C CNN
@@
 	7550 3250 7650 3250
 $Comp
-L MX_Alps_Hybrid:MX-NoLED MX2
+L MX_Alps_Hybrid:MX-NoLED MX3
 U 1 1 612C1DD8
 P 7100 3750
-F 0 "MX2" H 7133 3973 60  0000 C CNN
+F 0 "MX3" H 7133 3973 60  0000 C CNN
 F 1 "MX-NoLED" H 7133 3899 20  0000 C CNN
 F 2 "MX_Alps_Hybrid:MX-1U" H 6475 3725 60  0001 C CNN
@@
 $EndComp
 $Comp
-L Device:D_Small D2
+L Device:D_Small D3
 U 1 1 612C31B4
 P 6950 4000
-F 0 "D2" V 6996 3930 50  0000 R CNN
+F 0 "D3" V 6996 3930 50  0000 R CNN
 F 1 "SOD-123" V 6905 3930 50  0000 R CNN
 F 2 "Diode_SMD:D_SOD-123" V 6950 4000 50  0001 C CNN
@@
 Wire Wire Line
 	5850 1650 6000 1650
+Text GLabel 4100 2100 2    50   Input ~ 0
+COL1
+Text GLabel 4100 2200 2    50   Input ~ 0
+COL0
+Text GLabel 4100 2300 2    50   Input ~ 0
+ROW1
+Text GLabel 4100 3600 2    50   Input ~ 0
+ROW0
 $EndSCHEMATC
